File: gnss_receiver/hw/kicad/02_power.kicad_sch (KiCad schematic)
At the start: 59 parts

Commit message: МГП-8: КД в DOCX рядом с PDF; предприятие — ООО ШИВА НЕТВОРК
- tools/eskd_docx.py: выгрузка в DOCX по ЕСКД. Рамка и боковые графы — VML в
  колонтитуле за текстом, штамп форм 2/2а, osifont встроен, число листов — полями
  PAGE/NUMPAGES, выход детерминирован.
- ТЗ, ПЗ, ПМ, описание программы (build_docs.py) и ПЭ3, спецификация, ВП
  (eskd_lists.py) выходят в kd/ также в .docx. Подлинник — PDF, DOCX — редактируемая
  копия; правки вносятся в исходники.
- Перечни проверены в Word: число листов совпадает с PDF. Высота последней строки
  листа подобрана с запасом 1,2 мм до штампа (LIST_GAP).
- Предприятие в штампах всех документов и листов Э3 — «ООО ШИВА НЕТВОРК».
- Рамка Э3: надписи со знаком «№» набраны шрифтом osifont, потому что в штриховом
  шрифте KiCad этого знака нет.
- eskd_pdf.py: разбор md и размеры таблиц и рисунков вынесены в общие функции; PDF
  не изменился.
- README, CLAUDE.md: python-docx, порядок выгрузки DOCX, журнал передачи.

Co-Authored-By: Claude Opus 5.5 <noreply@anthropic.com>
Other:
- company: SiwaNetwork -> ООО ШИВА НЕТВОРК
Changed lines of the file:
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@@
     (date "08.10.2026")
     (rev "")
-    (company "SiwaNetwork")
+    (company "ООО ШИВА НЕТВОРК")
     (comment 1 "ШИВА.468157.001 Э3")
     (comment 2 "Разработчик")
