File: gnss_receiver/hw/kicad/05_rf2.kicad_sch (KiCad schematic)
At the start: 68 parts

Commit message: МГП-8: Э3 — нижний диапазон MAX2771 для каналов 3–8, сборка схемы на KiCad 10 (Windows)
Все восемь MAX2771 были включены через тракт верхнего диапазона (LNAIN_HI/MIXIN_HI,
согласование под 1575 МГц), хотя каналы 3–8 работают на 1176…1279 МГц. Каналы 3–8
переведены на LNAIN_LO/LNAOUT_LO/MIXIN_LO с согласованием 8,2 нГн + 1,1 пФ (у ADI —
8,4 нГн + 1,1 пФ), каналы 1–2 остались на верхнем (5,6 нГн + 1,7 пФ). Входы
неиспользуемого диапазона замкнуты на общий провод. ПЭ3, спецификация (9 листов), ВП,
Э3 пересобраны; ПЗ 4.2.4 (тракты и биты LNAMODE/MIXERMODE/LOBAND), 5.1.1 (Кш по диапазонам).

Генератор схемы работает на Windows с KiCad 10: поиск библиотеки УГО и шаблонов,
слой совместимости с библиотекой KiCad 7 (имена и номера выводов, порядок выводов) —
выход побайтно совпадает с KiCad 7. build.py --pdf выгружает Э3 через kicad-cli со
шрифтом osifont из tools/fonts (без установки в систему). build_docs: подсчёт листов
через pymupdf, если нет pypdf.

Co-Authored-By: Claude Opus 5.5 <noreply@anthropic.com>
Parts:
- C103, C116, C129, C93: value 1,7пФ -> 1,1пФ; Артикул GJM1555C1H1R7BB01D -> GJM1555C1H1R1BB01D; Наименование Конденсатор 0402 C0G 50 В 1,7 пФ -> Конденсатор 0402 C0G 50 В 1,1 пФ
- L10, L11, L8, L9: value 5,6нГн -> 8,2нГн; Артикул LQW15AN5N6C8ZD -> LQW15AN8N2G8ZD; Наименование Катушка индуктивности 0402 5,6 нГн ±0,2 нГн -> Катушка индуктивности 0402 8,2 нГн ±2 %
Connections:
- net GND: now also DA19.19 (LNAIN_HI), DA19.25 (MIXIN_HI), DA20.19 (LNAIN_HI), DA20.25 (MIXIN_HI), DA21.19 (LNAIN_HI), DA21.25 (MIXIN_HI), DA22.19 (LNAIN_HI), DA22.25 (MIXIN_HI); no longer DA19.20 (LNAIN_LO), DA19.26 (MIXIN_LO), DA20.20 (LNAIN_LO), DA20.26 (MIXIN_LO), DA21.20 (LNAIN_LO), DA21.26 (MIXIN_LO), DA22.20 (LNAIN_LO), DA22.26 (MIXIN_LO)
- net LNAIN_E: now also DA19.20 (LNAIN_LO); no longer DA19.19 (LNAIN_HI)
- net LNAIN_F: now also DA20.20 (LNAIN_LO); no longer DA20.19 (LNAIN_HI)
- net LNAIN_G: now also DA21.20 (LNAIN_LO); no longer DA21.19 (LNAIN_HI)
- net LNAIN_H: now also DA22.20 (LNAIN_LO); no longer DA22.19 (LNAIN_HI)
- net LNAO_E: now also DA19.23 (LNAOUT_LO); no longer DA19.24 (LNAOUT_HI)
- net LNAO_F: now also DA20.23 (LNAOUT_LO); no longer DA20.24 (LNAOUT_HI)
- net LNAO_G: now also DA21.23 (LNAOUT_LO); no longer DA21.24 (LNAOUT_HI)
- net LNAO_H: now also DA22.23 (LNAOUT_LO); no longer DA22.24 (LNAOUT_HI)
- net MIXI_E: now also DA19.26 (MIXIN_LO); no longer DA19.25 (MIXIN_HI)
- net MIXI_F: now also DA20.26 (MIXIN_LO); no longer DA20.25 (MIXIN_HI)
- net MIXI_G: now also DA21.26 (MIXIN_LO); no longer DA21.25 (MIXIN_HI)
- net MIXI_H: now also DA22.26 (MIXIN_LO); no longer DA22.25 (MIXIN_HI)

Commit message: МГП-8: КД в DOCX рядом с PDF; предприятие — ООО ШИВА НЕТВОРК
- tools/eskd_docx.py: выгрузка в DOCX по ЕСКД. Рамка и боковые графы — VML в
  колонтитуле за текстом, штамп форм 2/2а, osifont встроен, число листов — полями
  PAGE/NUMPAGES, выход детерминирован.
- ТЗ, ПЗ, ПМ, описание программы (build_docs.py) и ПЭ3, спецификация, ВП
  (eskd_lists.py) выходят в kd/ также в .docx. Подлинник — PDF, DOCX — редактируемая
  копия; правки вносятся в исходники.
- Перечни проверены в Word: число листов совпадает с PDF. Высота последней строки
  листа подобрана с запасом 1,2 мм до штампа (LIST_GAP).
- Предприятие в штампах всех документов и листов Э3 — «ООО ШИВА НЕТВОРК».
- Рамка Э3: надписи со знаком «№» набраны шрифтом osifont, потому что в штриховом
  шрифте KiCad этого знака нет.
- eskd_pdf.py: разбор md и размеры таблиц и рисунков вынесены в общие функции; PDF
  не изменился.
- README, CLAUDE.md: python-docx, порядок выгрузки DOCX, журнал передачи.

Co-Authored-By: Claude Opus 5.5 <noreply@anthropic.com>
Other:
- company: SiwaNetwork -> ООО ШИВА НЕТВОРК
Changed lines of the file:
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@@
     (date "08.10.2026")
     (rev "")
-    (company "SiwaNetwork")
+    (company "ООО ШИВА НЕТВОРК")
     (comment 1 "ШИВА.468157.001 Э3")
     (comment 2 "Разработчик")
