File: gnss_receiver/hw/kicad/10_usb.kicad_sch (KiCad schematic)
At the start: 48 parts, among them X4 M22-2510205

Commit message: МГП-8: навигационное ПО МК, расчёт мощности/надёжности, питание FX3 от импульсного стабилизатора, Э3 в КД
ПО МК (sw/fw):
- eph.c: координаты КА GPS/ГЛОНАСС/Galileo/BeiDou/QZSS (расхождение с эталоном < 0,4 мм)
- pvt.c: МНК по нескольким системам (отдельные шкалы), доплер -> скорость, DOP, тропосфера, Клобучар
- lnav.c: GPS LNAV — синхронизация, чётность, подкадры 1–3 и 4 (стр. 18), кодер для проверок
- rx.c: время излучения по границе подкадра и зеркалу NCO, псевдодальности, решение, момент 1PPS и qErr
- nmea.c: GGA, RMC, GSA, GSV, ZDA; rinex.c — чтение RINEX 3 (проверки на ПК)
- тесты: test_pvt (36 КА, 4 системы: 0,1 мм без шума), test_lnav (8 КА, обе полярности),
  test_rx_pvt (сквозной «ПЧ -> координаты, 1PPS», make test-long)

ПЛИС: копии счётчика слотов, расстояние до конца кода в LUTRAM, решение о новых шагах NCO
в стадии записи — движок 98–105 МГц, тесты движка и системы проходят.

Аппаратура: расчёт мощности выявил превышение 3,5 Вт в режиме USB 3.0 (4,03 Вт) из-за линейного
стабилизатора 5 -> 1,2 В ядра FX3; заменён на TPS62130, PG -> FX3_PWR_OK. Перестроены проект KiCad,
ПЭ3, спецификация, ВП; добавлен ШИВА.468157.001 Э3.pdf.
Расчёты: sim/power_budget.py (мощность, тепловой режим), sim/reliability.py (T0 ≈ 153 000 ч на борту БАС).
ТЗ: питание 5 В, питание антенны — перемычкой, ток 80 мА и программная защита, разводка порта времени.
tools/fix_osifont.py — воспроизводимое исправление шрифта.

Co-Authored-By: Claude Opus 5.5 <noreply@anthropic.com>
Claude-Session: https://claude.ai/code/session_011Z52gGMbqDGtKgZ2TDvqzY
Parts:
- added C234, C235: 100нФ, Capacitor_SMD:C_0402_1005Metric, symbol mgp8:C
- added L13: 2,2мкГн, Inductor_SMD:L_Coilcraft_XxL4020, symbol mgp8:L
- added R90: 49,9кОм, Resistor_SMD:R_0402_1005Metric, symbol mgp8:R
- added R91: 100кОм, Resistor_SMD:R_0402_1005Metric, symbol mgp8:R
- C223: value 22мкФ -> 10нФ; footprint Capacitor_SMD:C_0603_1608Metric -> Capacitor_SMD:C_0402_1005Metric; Артикул GRM188R61A226ME15D -> GRM155R71H103KA88D; Наименование Конденсатор 0603 X5R 10 В 22 мкФ -> Конденсатор 0402 X7R 50 В 10 нФ
- C224, C226: value 100нФ -> 10мкФ; footprint Capacitor_SMD:C_0402_1005Metric -> Capacitor_SMD:C_0603_1608Metric; Артикул GRM155R71C104KA88D -> GRM188R61A106KE69D; Наименование Конденсатор 0402 X7R 16 В 100 нФ -> Конденсатор 0603 X5R 10 В 10 мкФ
- C228: value 100нФ -> 10нФ; Артикул GRM155R71C104KA88D -> GRM155R71H103KA88D; Наименование Конденсатор 0402 X7R 16 В 100 нФ -> Конденсатор 0402 X7R 50 В 10 нФ
- C229: value 100нФ -> 22мкФ; footprint Capacitor_SMD:C_0402_1005Metric -> Capacitor_SMD:C_0603_1608Metric; Артикул GRM155R71C104KA88D -> GRM188R61A226ME15D; Наименование Конденсатор 0402 X7R 16 В 100 нФ -> Конденсатор 0603 X5R 10 В 22 мкФ
- C231, C233: value 10нФ -> 100нФ; Артикул GRM155R71H103KA88D -> GRM155R71C104KA88D; Наименование Конденсатор 0402 X7R 50 В 10 нФ -> Конденсатор 0402 X7R 16 В 100 нФ
- C232: value 10мкФ -> 100нФ; footprint Capacitor_SMD:C_0603_1608Metric -> Capacitor_SMD:C_0402_1005Metric; Артикул GRM188R61A106KE69D -> GRM155R71C104KA88D; Наименование Конденсатор 0603 X5R 10 В 10 мкФ -> Конденсатор 0402 X7R 16 В 100 нФ
- DA26: value USBLC6-2SC6 -> TPS62130RGTR; footprint Package_TO_SOT_SMD:SOT-23-6 -> Package_DFN_QFN:VQFN-16-1EP_3x3mm_P0.5mm_EP1.68x1.68mm_ThermalVias; symbol mgp8:USBLC6 -> mgp8:TPS62130; Артикул USBLC6-2SC6 -> TPS62130RGTR; Изготовитель STMicroelectronics -> Texas Instruments; Наименование Микросхема USBLC6-2SC6 -> Микросхема TPS62130RGTR
- DA27: value SPX3819M5-L-1-2/TR -> USBLC6-2SC6; footprint Package_TO_SOT_SMD:SOT-23-5 -> Package_TO_SOT_SMD:SOT-23-6; symbol mgp8:SPX3819_1.2 -> mgp8:USBLC6; Артикул SPX3819M5-L-1-2/TR -> USBLC6-2SC6; Изготовитель MaxLinear -> STMicroelectronics; Наименование Микросхема SPX3819M5-L-1-2/TR -> Микросхема USBLC6-2SC6
Connections:
- net +1V2_FX3: now also DA26.14 (VOS), L13.2, R90.1; no longer DA27.5 (OUT)
- net +3V3_FX3: now also C231.1, C232.1, C233.1, C234.1, C235.1; no longer C223.1, C224.1, C226.1, C227.1, C228.1
- net +5V_USB: now also C224.1, C226.1, C227.1, DA26.10 (VIN), DA26.11, DA26.12, DA26.13 (EN), DA27.5 (VBUS); no longer C232.1, DA26.5 (VBUS), DA27.1 (IN), DA27.3 (EN)
- net FX3_BP33: now also C223.1; no longer C231.1
- net FX3_PWR_OK: now also DA26.4 (PG)
- net GND: now also DA26.15 (GND), DA26.16, DA26.17, DA26.6, DA26.7 (FSW), DA26.8 (DEF), C234.2, C235.2, R91.2; no longer DA26.2 (GND)
- net USB_DM: now also DA27.3 (I/O2), DA27.4 (I/O2); no longer DA26.3 (I/O2), DA26.4 (I/O2)
- net USB_DP: now also DA27.1 (I/O1), DA27.6 (I/O1); no longer DA26.1 (I/O1), DA26.6 (I/O1)
- removed net FX3_BP12: C233.1, DA27.4 (BP)
- new net FB_1V2_FX3: DA26.5 (FB), R90.2, R91.1
- new net SS_1V2_FX3: C228.1, DA26.9 (SS/TR)
- new net SW_1V2_FX3: DA26.1 (SW), DA26.2, DA26.3, L13.1
Other:
- note added: "DA26: GND (GND) — выв. 6, 15, 16, 17"
- note added: "DA26: SW (SW_1V2_FX3) — выв. 1, 2, 3"
- note added: "DA26: VIN (+5V_USB) — выв. 10, 11, 12"
- note added: "DA27: I/O1 (USB_DP) — выв. 1, 6"
- note added: "DA27: I/O2 (USB_DM) — выв. 3, 4"
- note removed: "DA26: I/O1 (USB_DP) — выв. 1, 6"
- note removed: "DA26: I/O2 (USB_DM) — выв. 3, 4"
- moved on the sheet: C223, C224, C225, C226, C227, C228, C229, C230, C231, C232, C233, DA25

Commit message: МГП-8: КД в DOCX рядом с PDF; предприятие — ООО ШИВА НЕТВОРК
- tools/eskd_docx.py: выгрузка в DOCX по ЕСКД. Рамка и боковые графы — VML в
  колонтитуле за текстом, штамп форм 2/2а, osifont встроен, число листов — полями
  PAGE/NUMPAGES, выход детерминирован.
- ТЗ, ПЗ, ПМ, описание программы (build_docs.py) и ПЭ3, спецификация, ВП
  (eskd_lists.py) выходят в kd/ также в .docx. Подлинник — PDF, DOCX — редактируемая
  копия; правки вносятся в исходники.
- Перечни проверены в Word: число листов совпадает с PDF. Высота последней строки
  листа подобрана с запасом 1,2 мм до штампа (LIST_GAP).
- Предприятие в штампах всех документов и листов Э3 — «ООО ШИВА НЕТВОРК».
- Рамка Э3: надписи со знаком «№» набраны шрифтом osifont, потому что в штриховом
  шрифте KiCad этого знака нет.
- eskd_pdf.py: разбор md и размеры таблиц и рисунков вынесены в общие функции; PDF
  не изменился.
- README, CLAUDE.md: python-docx, порядок выгрузки DOCX, журнал передачи.

Co-Authored-By: Claude Opus 5.5 <noreply@anthropic.com>
Other:
- company: SiwaNetwork -> ООО ШИВА НЕТВОРК
Changed lines of the file:
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@@
     (date "08.10.2026")
     (rev "")
-    (company "SiwaNetwork")
+    (company "ООО ШИВА НЕТВОРК")
     (comment 1 "ШИВА.468157.001 Э3")
     (comment 2 "Разработчик")
