File: gnss_receiver/hw/kicad/11_io.kicad_sch (KiCad schematic)
At the start: 11 parts, among them X5 SM06B-GHS-TB, X6 SM04B-GHS-TB, X7 SM04B-GHS-TB, X8 SM04B-SRSS-TB

Commit message: МГП-8: навигационное ПО МК, расчёт мощности/надёжности, питание FX3 от импульсного стабилизатора, Э3 в КД
ПО МК (sw/fw):
- eph.c: координаты КА GPS/ГЛОНАСС/Galileo/BeiDou/QZSS (расхождение с эталоном < 0,4 мм)
- pvt.c: МНК по нескольким системам (отдельные шкалы), доплер -> скорость, DOP, тропосфера, Клобучар
- lnav.c: GPS LNAV — синхронизация, чётность, подкадры 1–3 и 4 (стр. 18), кодер для проверок
- rx.c: время излучения по границе подкадра и зеркалу NCO, псевдодальности, решение, момент 1PPS и qErr
- nmea.c: GGA, RMC, GSA, GSV, ZDA; rinex.c — чтение RINEX 3 (проверки на ПК)
- тесты: test_pvt (36 КА, 4 системы: 0,1 мм без шума), test_lnav (8 КА, обе полярности),
  test_rx_pvt (сквозной «ПЧ -> координаты, 1PPS», make test-long)

ПЛИС: копии счётчика слотов, расстояние до конца кода в LUTRAM, решение о новых шагах NCO
в стадии записи — движок 98–105 МГц, тесты движка и системы проходят.

Аппаратура: расчёт мощности выявил превышение 3,5 Вт в режиме USB 3.0 (4,03 Вт) из-за линейного
стабилизатора 5 -> 1,2 В ядра FX3; заменён на TPS62130, PG -> FX3_PWR_OK. Перестроены проект KiCad,
ПЭ3, спецификация, ВП; добавлен ШИВА.468157.001 Э3.pdf.
Расчёты: sim/power_budget.py (мощность, тепловой режим), sim/reliability.py (T0 ≈ 153 000 ч на борту БАС).
ТЗ: питание 5 В, питание антенны — перемычкой, ток 80 мА и программная защита, разводка порта времени.
tools/fix_osifont.py — воспроизводимое исправление шрифта.

Co-Authored-By: Claude Opus 5.5 <noreply@anthropic.com>
Claude-Session: https://claude.ai/code/session_011Z52gGMbqDGtKgZ2TDvqzY
Parts:
- removed R90, R91: 100Ом, Resistor_SMD:R_0402_1005Metric, symbol mgp8:R
- added R94, R95: 2,2кОм, Resistor_SMD:R_0402_1005Metric, symbol mgp8:R
- R92, R93: value 2,2кОм -> 100Ом; Артикул RC0402FR-072K2L -> RC0402FR-07100RL; Наименование Резистор 0402 2,2 кОм ±1 % 0,063 Вт -> Резистор 0402 100 Ом ±1 % 0,063 Вт; Примечание Подтяжка I2C, по заказу -> (none); now fitted; now in the parts list
Connections:
- net +3V3D: now also R94.1, R95.1; no longer R92.1, R93.1
- net GPS_P_RX: now also R92.1
- net GPS_P_TX: now also R93.1
- net GPS_RX: now also R92.2
- net GPS_SCL: now also R94.2; no longer R92.2
- net GPS_SDA: now also R95.2; no longer R93.2
- net GPS_TX: now also R93.2
Changed lines of the file:
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@@
     (on_board yes)
     (dnp no)
-    (property "Reference" "R90"
+    (property "Reference" "R92"
       (at 31.14 111.63 0)
       (effects
@@
       (project "mgp8"
         (path "/b897eb84-c3a6-5407-9ace-c16a4e8ba270/5f8847ce-ecb2-5f29-87ff-c0bcc04b90b9"
-          (reference "R90")
+          (reference "R92")
           (unit 1)
         )
@@
     (on_board yes)
     (dnp no)
-    (property "Reference" "R91"
+    (property "Reference" "R93"
       (at 48.92 111.63 0)
       (effects
@@
       (project "mgp8"
         (path "/b897eb84-c3a6-5407-9ace-c16a4e8ba270/5f8847ce-ecb2-5f29-87ff-c0bcc04b90b9"
-          (reference "R91")
+          (reference "R93")
           (unit 1)
         )
@@
     (on_board yes)
     (dnp yes)
-    (property "Reference" "R92"
+    (property "Reference" "R94"
       (at 67.97 105.28 0)
       (effects
@@
       (project "mgp8"
         (path "/b897eb84-c3a6-5407-9ace-c16a4e8ba270/5f8847ce-ecb2-5f29-87ff-c0bcc04b90b9"
-          (reference "R92")
+          (reference "R94")
           (unit 1)
         )
@@
     (on_board yes)
     (dnp yes)
-    (property "Reference" "R93"
+    (property "Reference" "R95"
       (at 90.83 105.28 0)
       (effects
@@
       (project "mgp8"
         (path "/b897eb84-c3a6-5407-9ace-c16a4e8ba270/5f8847ce-ecb2-5f29-87ff-c0bcc04b90b9"
-          (reference "R93")
+          (reference "R95")
           (unit 1)
         )

Commit message: МГП-8: КД в DOCX рядом с PDF; предприятие — ООО ШИВА НЕТВОРК
- tools/eskd_docx.py: выгрузка в DOCX по ЕСКД. Рамка и боковые графы — VML в
  колонтитуле за текстом, штамп форм 2/2а, osifont встроен, число листов — полями
  PAGE/NUMPAGES, выход детерминирован.
- ТЗ, ПЗ, ПМ, описание программы (build_docs.py) и ПЭ3, спецификация, ВП
  (eskd_lists.py) выходят в kd/ также в .docx. Подлинник — PDF, DOCX — редактируемая
  копия; правки вносятся в исходники.
- Перечни проверены в Word: число листов совпадает с PDF. Высота последней строки
  листа подобрана с запасом 1,2 мм до штампа (LIST_GAP).
- Предприятие в штампах всех документов и листов Э3 — «ООО ШИВА НЕТВОРК».
- Рамка Э3: надписи со знаком «№» набраны шрифтом osifont, потому что в штриховом
  шрифте KiCad этого знака нет.
- eskd_pdf.py: разбор md и размеры таблиц и рисунков вынесены в общие функции; PDF
  не изменился.
- README, CLAUDE.md: python-docx, порядок выгрузки DOCX, журнал передачи.

Co-Authored-By: Claude Opus 5.5 <noreply@anthropic.com>
Other:
- company: SiwaNetwork -> ООО ШИВА НЕТВОРК
Changed lines of the file:
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@@
     (date "08.10.2026")
     (rev "")
-    (company "SiwaNetwork")
+    (company "ООО ШИВА НЕТВОРК")
     (comment 1 "ШИВА.468157.001 Э3")
     (comment 2 "Разработчик")
