File: gnss_receiver/hw/kicad/08_fpga2.kicad_sch (KiCad schematic)
At the start: 53 parts, among them X1 FTSH-105-01-L-DV-K, X2 FTSH-105-01-L-DV-K

Commit message: МГП-8: КД в DOCX рядом с PDF; предприятие — ООО ШИВА НЕТВОРК
- tools/eskd_docx.py: выгрузка в DOCX по ЕСКД. Рамка и боковые графы — VML в
  колонтитуле за текстом, штамп форм 2/2а, osifont встроен, число листов — полями
  PAGE/NUMPAGES, выход детерминирован.
- ТЗ, ПЗ, ПМ, описание программы (build_docs.py) и ПЭ3, спецификация, ВП
  (eskd_lists.py) выходят в kd/ также в .docx. Подлинник — PDF, DOCX — редактируемая
  копия; правки вносятся в исходники.
- Перечни проверены в Word: число листов совпадает с PDF. Высота последней строки
  листа подобрана с запасом 1,2 мм до штампа (LIST_GAP).
- Предприятие в штампах всех документов и листов Э3 — «ООО ШИВА НЕТВОРК».
- Рамка Э3: надписи со знаком «№» набраны шрифтом osifont, потому что в штриховом
  шрифте KiCad этого знака нет.
- eskd_pdf.py: разбор md и размеры таблиц и рисунков вынесены в общие функции; PDF
  не изменился.
- README, CLAUDE.md: python-docx, порядок выгрузки DOCX, журнал передачи.

Co-Authored-By: Claude Opus 5.5 <noreply@anthropic.com>
Other:
- company: SiwaNetwork -> ООО ШИВА НЕТВОРК
Changed lines of the file:
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@@
     (date "08.10.2026")
     (rev "")
-    (company "SiwaNetwork")
+    (company "ООО ШИВА НЕТВОРК")
     (comment 1 "ШИВА.468157.001 Э3")
     (comment 2 "Разработчик")

Commit message: МГП-8: печатная плата в KiCad, габариты и масса, тепловая модель платы
- hw/gen/pcb.py, pcb_place.py: плата 100×75 мм, 8 слоёв (L2/L4/L7 — земля,
  L5 — островки питания), размещение по узлам схемы, RF и тактовые цепи —
  сценарием (ВЧ-входы по 47,17 мм, ADC_CLK по 58,99 мм), остальное —
  Freerouting 2.5; переходы к слоям земли/питания, заливки, DRC;
- hw/gen/footprints.py → hw/kicad/mgp8.pretty, правила mgp8.kicad_dru;
  в генераторе схемы — имена посадочных мест по библиотеке KiCad 10,
  blocks.json для размещения, kicad_pro сохраняет правила платы;
- DRC KiCad 10: ошибок нет, схема и плата совпадают; не разведено
  161 соединение из 1140 — довести вручную (ПЗ 9.1, п. 1);
- sim/mech_budget.py: высота 9,90 мм (≤ 12), масса 56,7 г (≤ 80);
- sim/thermal_board.py: тепловая модель платы при +85 °С, Tj ПЛИС, МК
  и FX3 не выше 92,8 °С с отводом на крышку корпуса;
- ПЗ 4.7, 5.7, таблица 5, 9.1; КД (ПЗ, ЭП) пересобрана; CLAUDE.md.

Co-Authored-By: Claude Opus 5.5 <noreply@anthropic.com>
Parts:
- DD7: footprint Package_BGA:Lattice_caBGA-381_17.0x17.0mm_Layout20x20_P0.8mm_Ball0.4mm_Pad0.4mm_NSMD -> Package_BGA:Lattice_caBGA-381_17x17mm_Layout20x20_P0.8mm
- DD8: footprint Package_SO:SOIC-8_5.23x5.23mm_P1.27mm -> Package_SO:SOIC-8_5.3x5.3mm_P1.27mm
Changed lines of the file:
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@@
       )
     )
-    (property "Footprint" "Package_BGA:Lattice_caBGA-381_17.0x17.0mm_Layout20x20_P0.8mm_Ball0.4mm_Pad0.4mm_NSMD"
+    (property "Footprint" "Package_BGA:Lattice_caBGA-381_17x17mm_Layout20x20_P0.8mm"
       (at 88.9 83.82 0)
       (effects
@@
       )
     )
-    (property "Footprint" "Package_BGA:Lattice_caBGA-381_17.0x17.0mm_Layout20x20_P0.8mm_Ball0.4mm_Pad0.4mm_NSMD"
+    (property "Footprint" "Package_BGA:Lattice_caBGA-381_17x17mm_Layout20x20_P0.8mm"
       (at 194.31 73.66 0)
       (effects
@@
       )
     )
-    (property "Footprint" "Package_SO:SOIC-8_5.23x5.23mm_P1.27mm"
+    (property "Footprint" "Package_SO:SOIC-8_5.3x5.3mm_P1.27mm"
       (at 279.4 63.5 0)
       (effects
