File: gnss_receiver/hw/kicad/07_fpga1.kicad_sch (KiCad schematic)
At the start: 1 part

Commit message: МГП-8: КД в DOCX рядом с PDF; предприятие — ООО ШИВА НЕТВОРК
- tools/eskd_docx.py: выгрузка в DOCX по ЕСКД. Рамка и боковые графы — VML в
  колонтитуле за текстом, штамп форм 2/2а, osifont встроен, число листов — полями
  PAGE/NUMPAGES, выход детерминирован.
- ТЗ, ПЗ, ПМ, описание программы (build_docs.py) и ПЭ3, спецификация, ВП
  (eskd_lists.py) выходят в kd/ также в .docx. Подлинник — PDF, DOCX — редактируемая
  копия; правки вносятся в исходники.
- Перечни проверены в Word: число листов совпадает с PDF. Высота последней строки
  листа подобрана с запасом 1,2 мм до штампа (LIST_GAP).
- Предприятие в штампах всех документов и листов Э3 — «ООО ШИВА НЕТВОРК».
- Рамка Э3: надписи со знаком «№» набраны шрифтом osifont, потому что в штриховом
  шрифте KiCad этого знака нет.
- eskd_pdf.py: разбор md и размеры таблиц и рисунков вынесены в общие функции; PDF
  не изменился.
- README, CLAUDE.md: python-docx, порядок выгрузки DOCX, журнал передачи.

Co-Authored-By: Claude Opus 5.5 <noreply@anthropic.com>
Other:
- company: SiwaNetwork -> ООО ШИВА НЕТВОРК
Changed lines of the file:
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@@
     (date "08.10.2026")
     (rev "")
-    (company "SiwaNetwork")
+    (company "ООО ШИВА НЕТВОРК")
     (comment 1 "ШИВА.468157.001 Э3")
     (comment 2 "Разработчик")

Commit message: МГП-8: печатная плата в KiCad, габариты и масса, тепловая модель платы
- hw/gen/pcb.py, pcb_place.py: плата 100×75 мм, 8 слоёв (L2/L4/L7 — земля,
  L5 — островки питания), размещение по узлам схемы, RF и тактовые цепи —
  сценарием (ВЧ-входы по 47,17 мм, ADC_CLK по 58,99 мм), остальное —
  Freerouting 2.5; переходы к слоям земли/питания, заливки, DRC;
- hw/gen/footprints.py → hw/kicad/mgp8.pretty, правила mgp8.kicad_dru;
  в генераторе схемы — имена посадочных мест по библиотеке KiCad 10,
  blocks.json для размещения, kicad_pro сохраняет правила платы;
- DRC KiCad 10: ошибок нет, схема и плата совпадают; не разведено
  161 соединение из 1140 — довести вручную (ПЗ 9.1, п. 1);
- sim/mech_budget.py: высота 9,90 мм (≤ 12), масса 56,7 г (≤ 80);
- sim/thermal_board.py: тепловая модель платы при +85 °С, Tj ПЛИС, МК
  и FX3 не выше 92,8 °С с отводом на крышку корпуса;
- ПЗ 4.7, 5.7, таблица 5, 9.1; КД (ПЗ, ЭП) пересобрана; CLAUDE.md.

Co-Authored-By: Claude Opus 5.5 <noreply@anthropic.com>
Parts:
- DD7: footprint Package_BGA:Lattice_caBGA-381_17.0x17.0mm_Layout20x20_P0.8mm_Ball0.4mm_Pad0.4mm_NSMD -> Package_BGA:Lattice_caBGA-381_17x17mm_Layout20x20_P0.8mm
Changed lines of the file:
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@@
       )
     )
-    (property "Footprint" "Package_BGA:Lattice_caBGA-381_17.0x17.0mm_Layout20x20_P0.8mm_Ball0.4mm_Pad0.4mm_NSMD"
+    (property "Footprint" "Package_BGA:Lattice_caBGA-381_17x17mm_Layout20x20_P0.8mm"
       (at 76.2 78.74 0)
       (effects
@@
       )
     )
-    (property "Footprint" "Package_BGA:Lattice_caBGA-381_17.0x17.0mm_Layout20x20_P0.8mm_Ball0.4mm_Pad0.4mm_NSMD"
+    (property "Footprint" "Package_BGA:Lattice_caBGA-381_17x17mm_Layout20x20_P0.8mm"
       (at 191.77 83.82 0)
       (effects
@@
       )
     )
-    (property "Footprint" "Package_BGA:Lattice_caBGA-381_17.0x17.0mm_Layout20x20_P0.8mm_Ball0.4mm_Pad0.4mm_NSMD"
+    (property "Footprint" "Package_BGA:Lattice_caBGA-381_17x17mm_Layout20x20_P0.8mm"
       (at 302.26 83.82 0)
       (effects
@@
       )
     )
-    (property "Footprint" "Package_BGA:Lattice_caBGA-381_17.0x17.0mm_Layout20x20_P0.8mm_Ball0.4mm_Pad0.4mm_NSMD"
+    (property "Footprint" "Package_BGA:Lattice_caBGA-381_17x17mm_Layout20x20_P0.8mm"
       (at 394.97 83.82 0)
       (effects
@@
       )
     )
-    (property "Footprint" "Package_BGA:Lattice_caBGA-381_17.0x17.0mm_Layout20x20_P0.8mm_Ball0.4mm_Pad0.4mm_NSMD"
+    (property "Footprint" "Package_BGA:Lattice_caBGA-381_17x17mm_Layout20x20_P0.8mm"
       (at 482.6 83.82 0)
       (effects
@@
       )
     )
-    (property "Footprint" "Package_BGA:Lattice_caBGA-381_17.0x17.0mm_Layout20x20_P0.8mm_Ball0.4mm_Pad0.4mm_NSMD"
+    (property "Footprint" "Package_BGA:Lattice_caBGA-381_17x17mm_Layout20x20_P0.8mm"
       (at 73.66 196.85 0)
       (effects

Commit message: МГП-8: плата разведена полностью — 0 неразведённых соединений, DRC без ошибок
- Выводы каналов MAX2771 на ПЛИС переназначены по положению на плате: каналы 5–8 —
  банк 7, 1–4 — банк 6, шины над ПЛИС не пересекаются (design.py, mgp8.lpf,
  fpga_pinout.json, лист 07_fpga1, Э3).
- ПЛИС пересобрана: 100,15 МГц (вес тайминга при размещении — PNR в Makefile).
- Доразводка: совместные отводы нижнего ряда MAX2771, обход XTAL_A, вложенная перекладка
  с откатом. Проводников 9303, переходов 1320, 10,65 м; DRC — ошибок 0, расхождений со
  схемой 0, неразведённых 0 (предупреждения: 14 висящих отрезков, 9 переходов, 3 наложения
  шелкографии).
- Пересчитаны масса (55,9 г) и тепловая модель (Tj ПЛИС/МК/FX3 ≤ 92,7 °С); ПЗ 4.7.4,
  4.7.5, 5.7.2, 6.2.2, табл. 5, 9.1; КД пересобрана.

Co-Authored-By: Claude Opus 5.5 <noreply@anthropic.com>
Connections:
- net MAX_CSN_A: now also DD7.P1; no longer DD7.B2
- net MAX_CSN_B: now also DD7.M4; no longer DD7.C4
- net MAX_CSN_C: now also DD7.L1; no longer DD7.E2 (E2 PCLKC7_0)
- net MAX_CSN_D: now also DD7.J4 (J4 GR_PCLK6_0); no longer DD7.F5
- net MAX_CSN_E: now also DD7.F5; no longer DD7.J4 (J4 GR_PCLK6_0)
- net MAX_CSN_F: now also DD7.E2 (E2 PCLKC7_0); no longer DD7.L1
- net MAX_CSN_G: now also DD7.C4; no longer DD7.M4
- net MAX_CSN_H: now also DD7.B2; no longer DD7.P1
- net MAX_I0_A: now also DD7.N2; no longer DD7.A3
- net MAX_I0_B: now also DD7.L4; no longer DD7.B5
- net MAX_I0_C: now also DD7.K2; no longer DD7.D2
- net MAX_I0_D: now also DD7.G1 (G1 PCLKC6_0); no longer DD7.E5
- net MAX_I0_E: now also DD7.E5; no longer DD7.G1 (G1 PCLKC6_0)
- net MAX_I0_F: now also DD7.D2; no longer DD7.K2
- net MAX_I0_G: now also DD7.B5; no longer DD7.L4
- net MAX_I0_H: now also DD7.A3; no longer DD7.N2
- net MAX_I1_A: now also DD7.N1; no longer DD7.A2
- net MAX_I1_B: now also DD7.L3; no longer DD7.B4
- net MAX_I1_C: now also DD7.K1; no longer DD7.D1
- net MAX_I1_D: now also DD7.F1 (F1 PCLKC6_1); no longer DD7.E4
- net MAX_I1_E: now also DD7.E4; no longer DD7.F1 (F1 PCLKC6_1)
- net MAX_I1_F: now also DD7.D1; no longer DD7.K1
- net MAX_I1_G: now also DD7.B4; no longer DD7.L3
- net MAX_I1_H: now also DD7.A2; no longer DD7.N1
- net MAX_LD_A: now also DD7.N5; no longer DD7.B1
- net MAX_LD_B: now also DD7.M3; no longer DD7.C3
- net MAX_LD_C: now also DD7.K5; no longer DD7.E1
- net MAX_LD_D: now also DD7.J3 (J3 GR_PCLK6_1); no longer DD7.F4
- net MAX_LD_E: now also DD7.F4; no longer DD7.J3 (J3 GR_PCLK6_1)
- net MAX_LD_F: now also DD7.E1; no longer DD7.K5
- net MAX_LD_G: now also DD7.C3; no longer DD7.M3
- net MAX_LD_H: now also DD7.B1; no longer DD7.N5
- net MAX_Q0_A: now also DD7.N4; no longer DD7.A5
- net MAX_Q0_B: now also DD7.M1; no longer DD7.C2
- net MAX_Q0_C: now also DD7.K4; no longer DD7.D5
- net MAX_Q0_D: now also DD7.J1; no longer DD7.F3 (F3 PCLKC7_1)
- net MAX_Q0_E: now also DD7.F3 (F3 PCLKC7_1); no longer DD7.J1
- net MAX_Q0_F: now also DD7.D5; no longer DD7.K4
- net MAX_Q0_G: now also DD7.C2; no longer DD7.M1
- net MAX_Q0_H: now also DD7.A5; no longer DD7.N4
- net MAX_Q1_A: now also DD7.N3; no longer DD7.A4
- net MAX_Q1_B: now also DD7.L5; no longer DD7.C1
- net MAX_Q1_C: now also DD7.K3; no longer DD7.D3
- net MAX_Q1_D: now also DD7.H1; no longer DD7.F2 (F2 PCLKT7_0)
- net MAX_Q1_E: now also DD7.F2 (F2 PCLKT7_0); no longer DD7.H1
- net MAX_Q1_F: now also DD7.D3; no longer DD7.K3
- net MAX_Q1_G: now also DD7.C1; no longer DD7.L5
- net MAX_Q1_H: now also DD7.A4; no longer DD7.N3
- net MAX_SHDN_A: now also DD7.P2; no longer DD7.B3
- net MAX_SHDN_B: now also DD7.M5; no longer DD7.C5
- net MAX_SHDN_C: now also DD7.L2; no longer DD7.E3
- net MAX_SHDN_D: now also DD7.J5; no longer DD7.G3 (G3 PCLKT7_1)
- net MAX_SHDN_E: now also DD7.G3 (G3 PCLKT7_1); no longer DD7.J5
- net MAX_SHDN_F: now also DD7.E3; no longer DD7.L2
- net MAX_SHDN_G: now also DD7.C5; no longer DD7.M5
- net MAX_SHDN_H: now also DD7.B3; no longer DD7.P2
Changed lines of the file:
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@@
     )
   )
-  (global_label "MAX_I1_E"
+  (global_label "MAX_I1_D"
     (shape bidirectional)
     (at 454.66 43.18 180)
@@
     )
   )
-  (global_label "MAX_I0_E"
+  (global_label "MAX_I0_D"
     (shape bidirectional)
     (at 454.66 48.26 180)
@@
     )
   )
-  (global_label "MAX_Q1_E"
+  (global_label "MAX_Q1_D"
     (shape bidirectional)
     (at 454.66 58.42 180)
@@
     )
   )
-  (global_label "MAX_Q0_E"
+  (global_label "MAX_Q0_D"
     (shape bidirectional)
     (at 454.66 68.58 180)
@@
     )
   )
-  (global_label "MAX_LD_E"
+  (global_label "MAX_LD_D"
     (shape bidirectional)
     (at 454.66 73.66 180)
@@
     )
   )
-  (global_label "MAX_CSN_E"
+  (global_label "MAX_CSN_D"
     (shape bidirectional)
     (at 454.66 78.74 180)
@@
     )
   )
-  (global_label "MAX_SHDN_E"
+  (global_label "MAX_SHDN_D"
     (shape bidirectional)
     (at 454.66 83.82 180)
@@
     )
   )
-  (global_label "MAX_I1_F"
+  (global_label "MAX_I1_C"
     (shape bidirectional)
     (at 454.66 88.9 180)
@@
     )
   )
-  (global_label "MAX_I0_F"
+  (global_label "MAX_I0_C"
     (shape bidirectional)
     (at 454.66 93.98 180)
@@
     )
   )
-  (global_label "MAX_Q1_F"
+  (global_label "MAX_Q1_C"
     (shape bidirectional)
     (at 454.66 99.06 180)
@@
     )
   )
-  (global_label "MAX_Q0_F"
+  (global_label "MAX_Q0_C"
     (shape bidirectional)
     (at 454.66 104.14 180)
@@
     )
   )
-  (global_label "MAX_LD_F"
+  (global_label "MAX_LD_C"
     (shape bidirectional)
     (at 454.66 109.22 180)
@@
     )
   )
-  (global_label "MAX_CSN_F"
+  (global_label "MAX_CSN_C"
     (shape bidirectional)
     (at 454.66 114.3 180)
@@
     )
   )
-  (global_label "MAX_SHDN_F"
+  (global_label "MAX_SHDN_C"
     (shape bidirectional)
     (at 454.66 119.38 180)
@@
     )
   )
-  (global_label "MAX_I1_G"
+  (global_label "MAX_I1_B"
     (shape bidirectional)
     (at 454.66 124.46 180)
@@
     )
   )
-  (global_label "MAX_I0_G"
+  (global_label "MAX_I0_B"
     (shape bidirectional)
     (at 510.54 43.18 0)
@@
     )
   )
-  (global_label "MAX_Q1_G"
+  (global_label "MAX_Q1_B"
     (shape bidirectional)
     (at 510.54 48.26 0)
@@
     )
   )
-  (global_label "MAX_Q0_G"
+  (global_label "MAX_Q0_B"
     (shape bidirectional)
     (at 510.54 53.34 0)
@@
     )
   )
-  (global_label "MAX_LD_G"
+  (global_label "MAX_LD_B"
     (shape bidirectional)
     (at 510.54 58.42 0)
@@
     )
   )
-  (global_label "MAX_CSN_G"
+  (global_label "MAX_CSN_B"
     (shape bidirectional)
     (at 510.54 63.5 0)
@@
     )
   )
-  (global_label "MAX_SHDN_G"
+  (global_label "MAX_SHDN_B"
     (shape bidirectional)
     (at 510.54 68.58 0)
@@
     )
   )
-  (global_label "MAX_I1_H"
+  (global_label "MAX_I1_A"
     (shape bidirectional)
     (at 510.54 73.66 0)
@@
     )
   )
-  (global_label "MAX_I0_H"
+  (global_label "MAX_I0_A"
     (shape bidirectional)
     (at 510.54 78.74 0)
@@
     )
   )
-  (global_label "MAX_Q1_H"
+  (global_label "MAX_Q1_A"
     (shape bidirectional)
     (at 510.54 83.82 0)
@@
     )
   )
-  (global_label "MAX_Q0_H"
+  (global_label "MAX_Q0_A"
     (shape bidirectional)
     (at 510.54 88.9 0)
@@
     )
   )
-  (global_label "MAX_LD_H"
+  (global_label "MAX_LD_A"
     (shape bidirectional)
     (at 510.54 93.98 0)
@@
     )
   )
-  (global_label "MAX_CSN_H"
+  (global_label "MAX_CSN_A"
     (shape bidirectional)
     (at 510.54 99.06 0)
@@
     )
   )
-  (global_label "MAX_SHDN_H"
+  (global_label "MAX_SHDN_A"
     (shape bidirectional)
     (at 510.54 104.14 0)
@@
     )
   )
-  (global_label "MAX_I1_A"
+  (global_label "MAX_I1_H"
     (shape bidirectional)
     (at 45.72 156.21 180)
@@
     )
   )
-  (global_label "MAX_I0_A"
+  (global_label "MAX_I0_H"
     (shape bidirectional)
     (at 45.72 161.29 180)
@@
     )
   )
-  (global_label "MAX_Q1_A"
+  (global_label "MAX_Q1_H"
     (shape bidirectional)
     (at 45.72 166.37 180)
@@
     )
   )
-  (global_label "MAX_Q0_A"
+  (global_label "MAX_Q0_H"
     (shape bidirectional)
     (at 45.72 171.45 180)
@@
     )
   )
-  (global_label "MAX_LD_A"
+  (global_label "MAX_LD_H"
     (shape bidirectional)
     (at 45.72 176.53 180)
@@
     )
   )
-  (global_label "MAX_CSN_A"
+  (global_label "MAX_CSN_H"
     (shape bidirectional)
     (at 45.72 181.61 180)
@@
     )
   )
-  (global_label "MAX_SHDN_A"
+  (global_label "MAX_SHDN_H"
     (shape bidirectional)
     (at 45.72 186.69 180)
@@
     )
   )
-  (global_label "MAX_I1_B"
+  (global_label "MAX_I1_G"
     (shape bidirectional)
     (at 45.72 191.77 180)
@@
     )
   )
-  (global_label "MAX_I0_B"
+  (global_label "MAX_I0_G"
     (shape bidirectional)
     (at 45.72 196.85 180)
@@
     )
   )
-  (global_label "MAX_Q1_B"
+  (global_label "MAX_Q1_G"
     (shape bidirectional)
     (at 45.72 201.93 180)
@@
     )
   )
-  (global_label "MAX_Q0_B"
+  (global_label "MAX_Q0_G"
     (shape bidirectional)
     (at 45.72 207.01 180)
@@
     )
   )
-  (global_label "MAX_LD_B"
+  (global_label "MAX_LD_G"
     (shape bidirectional)
     (at 45.72 212.09 180)
@@
     )
   )
-  (global_label "MAX_CSN_B"
+  (global_label "MAX_CSN_G"
     (shape bidirectional)
     (at 45.72 217.17 180)
@@
     )
   )
-  (global_label "MAX_SHDN_B"
+  (global_label "MAX_SHDN_G"
     (shape bidirectional)
     (at 45.72 222.25 180)
@@
     )
   )
-  (global_label "MAX_I1_C"
+  (global_label "MAX_I1_F"
     (shape bidirectional)
     (at 45.72 227.33 180)
@@
     )
   )
-  (global_label "MAX_I0_C"
+  (global_label "MAX_I0_F"
     (shape bidirectional)
     (at 45.72 232.41 180)
@@
     )
   )
-  (global_label "MAX_Q1_C"
+  (global_label "MAX_Q1_F"
     (shape bidirectional)
     (at 101.6 156.21 0)
@@
     )
   )
-  (global_label "MAX_Q0_C"
+  (global_label "MAX_Q0_F"
     (shape bidirectional)
     (at 101.6 161.29 0)
@@
     )
   )
-  (global_label "MAX_LD_C"
+  (global_label "MAX_LD_F"
     (shape bidirectional)
     (at 101.6 166.37 0)
@@
     )
   )
-  (global_label "MAX_CSN_C"
+  (global_label "MAX_CSN_F"
     (shape bidirectional)
     (at 101.6 171.45 0)
@@
     )
   )
-  (global_label "MAX_SHDN_C"
+  (global_label "MAX_SHDN_F"
     (shape bidirectional)
     (at 101.6 176.53 0)
@@
     )
   )
-  (global_label "MAX_I1_D"
+  (global_label "MAX_I1_E"
     (shape bidirectional)
     (at 101.6 181.61 0)
@@
     )
   )
-  (global_label "MAX_I0_D"
+  (global_label "MAX_I0_E"
     (shape bidirectional)
     (at 101.6 186.69 0)
@@
     )
   )
-  (global_label "MAX_Q1_D"
+  (global_label "MAX_Q1_E"
     (shape bidirectional)
     (at 101.6 191.77 0)
@@
     )
   )
-  (global_label "MAX_Q0_D"
+  (global_label "MAX_Q0_E"
     (shape bidirectional)
     (at 101.6 196.85 0)
@@
     )
   )
-  (global_label "MAX_LD_D"
+  (global_label "MAX_LD_E"
     (shape bidirectional)
     (at 101.6 201.93 0)
@@
     )
   )
-  (global_label "MAX_CSN_D"
+  (global_label "MAX_CSN_E"
     (shape bidirectional)
     (at 101.6 207.01 0)
@@
     )
   )
-  (global_label "MAX_SHDN_D"
+  (global_label "MAX_SHDN_E"
     (shape bidirectional)
     (at 101.6 212.09 0)
